File: Flex PCB 10by10 button array 1mm edge spacing copy/Flex PCB 10by10 button array 1mm.kicad_pcb (KiCad board)
At the start: 2 copper layers, 202 parts, among them J1 522071060, J2 522071060

Commit message: Add files via upload
Other:
- board outline added: 63.3 x 53.8 mm
- board text added: "Read"
- board text added: "Scan"
Changed lines of the file:
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@@
 		(embedded_fonts no)
+	)
+	(gr_circle
+		(center 220.3 98.1)
+		(end 221.95 98.1)
+		(stroke
+			(width 0.05)
+			(type solid)
+		)
+		(fill no)
+		(layer "Edge.Cuts")
+	)
+	(gr_circle
+		(center 218.3 70)
+		(end 219.95 70)
+		(stroke
+			(width 0.05)
+			(type solid)
+		)
+		(fill no)
+		(layer "Edge.Cuts")
+	)
+	(gr_circle
+		(center 164 70)
+		(end 165.65 70)
+		(stroke
+			(width 0.05)
+			(type solid)
+		)
+		(fill no)
+		(layer "Edge.Cuts")
+	)
+	(gr_rect
+		(start 159.35 67.35)
+		(end 222.7 121.15)
+		(stroke
+			(width 0.05)
+			(type default)
+		)
+		(fill no)
+		(layer "Edge.Cuts")
+	)
+	(gr_circle
+		(center 162 98.1)
+		(end 163.65 98.1)
+		(stroke
+			(width 0.05)
+			(type solid)
+		)
+		(fill no)
+		(layer "Edge.Cuts")
+	)
+	(gr_text "Scan"
+		(at 214.65 119.4 0)
+		(layer "F.SilkS")
+		(effects
+			(font
+				(size 1.5 1.5)
+				(thickness 0.3)
+				(bold yes)
+			)
+			(justify left bottom)
+		)
+	)
+	(gr_text "Read"
+		(at 162.95 119.75 0)
+		(layer "F.SilkS")
+		(effects
+			(font
+				(size 1.5 1.5)
+				(thickness 0.3)
+				(bold yes)
+			)
+			(justify left bottom)
+		)
 	)
 	(via
