File: COPY OF Flex PCB 10by10 button array 1mm edge spacing copy/Flex PCB 10by10 button array 1mm.kicad_pcb (KiCad board)
At the start: 2 copper layers, 69.7 x 153.1 mm, 202 parts, among them J1 522071060, J2 522071060

Commit message: Add files via upload
Parts:
- J1, J2: value 522071060 -> Conn_01x24; footprint costumized ffc connector 24pos:customized 24pos connector 1mm pitch footprint -> costumized ffc connector 24pos:24pos edge connector
Connections:
- J1 pad 11: (no net) -> unconnected-(J1-Pin_11-Pad11)
- J1 pad 12: (no net) -> unconnected-(J1-Pin_12-Pad12)
- J1 pad 13: (no net) -> unconnected-(J1-Pin_13-Pad13)
- J1 pad 14: (no net) -> unconnected-(J1-Pin_14-Pad14)
- J1 pad 15: (no net) -> unconnected-(J1-Pin_15-Pad15)
- J1 pad 16: (no net) -> unconnected-(J1-Pin_16-Pad16)
- J1 pad 17: (no net) -> unconnected-(J1-Pin_17-Pad17)
- J1 pad 18: (no net) -> unconnected-(J1-Pin_18-Pad18)
- J1 pad 19: (no net) -> unconnected-(J1-Pin_19-Pad19)
- J1 pad 20: (no net) -> unconnected-(J1-Pin_20-Pad20)
- J1 pad 21: (no net) -> unconnected-(J1-Pin_21-Pad21)
- J1 pad 22: (no net) -> unconnected-(J1-Pin_22-Pad22)
- J1 pad 23: (no net) -> unconnected-(J1-Pin_23-Pad23)
- J1 pad 24: (no net) -> unconnected-(J1-Pin_24-Pad24)
- J2 pad 11: (no net) -> unconnected-(J2-Pin_11-Pad11)
- J2 pad 12: (no net) -> unconnected-(J2-Pin_12-Pad12)
- J2 pad 13: (no net) -> unconnected-(J2-Pin_13-Pad13)
- J2 pad 14: (no net) -> unconnected-(J2-Pin_14-Pad14)
- J2 pad 15: (no net) -> unconnected-(J2-Pin_15-Pad15)
- J2 pad 16: (no net) -> unconnected-(J2-Pin_16-Pad16)
- J2 pad 17: (no net) -> unconnected-(J2-Pin_17-Pad17)
- J2 pad 18: (no net) -> unconnected-(J2-Pin_18-Pad18)
- J2 pad 19: (no net) -> unconnected-(J2-Pin_19-Pad19)
- J2 pad 20: (no net) -> unconnected-(J2-Pin_20-Pad20)
- J2 pad 21: (no net) -> unconnected-(J2-Pin_21-Pad21)
- J2 pad 22: (no net) -> unconnected-(J2-Pin_22-Pad22)
- J2 pad 23: (no net) -> unconnected-(J2-Pin_23-Pad23)
- J2 pad 24: (no net) -> unconnected-(J2-Pin_24-Pad24)
Routing:
- net Net-(J2-Pin_10): track 199.9 -> 200.7 mm
Other:
- board size 69.7 x 153.1 mm -> 68.7 x 152.8 mm
